Commit message: fixed lidar.. working properly now and can ve visualised in RViz

File: install/rcup_garden/share/rcup_garden/urdf/ArmPlate.urdf.xacro (robot description, xacro)
@@ -257,15 +257,9 @@
     <!-- WHEEL LINKS ENDS-->
     <!-- Updated part for correcting bot orientation on spawn -->
-    <link name="base_footprint">
-        <inertial>
-            <origin xyz="0.0 0.0 0.0" rpy="0.0 0.0 0.0" />
-            <mass value="56.0" />
-            <inertia ixx="2.5" iyy="2.5" izz="4.5" ixy="0.0" iyz="0.0" ixz="0.0" />
-        </inertial>
-    </link>
+    <link name="base_footprint"/>
     <joint name="base_to_robot" type="fixed">
-        <origin xyz="0.0 0.35 -0.07" rpy="1.57 0.0 1.57" />
-        <parent link="base_footprint" />
-        <child link="base_final-v3" />
+    <origin xyz="0.0 0.35 -0.07" rpy="1.57 0.0 1.57" />
+    <parent link="base_footprint" />
+    <child link="base_final-v3" />
     </joint>
     <gazebo reference="base_footprint">
@@ -1516,5 +1510,5 @@
     <gazebo reference="LIDAR_1-v1">
         <sensor name="lidar_sensor" type="gpu_lidar">
-            <pose>0 0 0 0 0 0</pose>
+            <pose>0 0 0 0 0 -1.5708</pose>
             <always_on>true</always_on>
             <visualize>true</visualize>
@@ -1525,6 +1519,6 @@
                         <samples>360</samples>
                         <resolution>1</resolution>
-                        <min_angle>-3.14</min_angle>
-                        <max_angle>0</max_angle>
+                        <min_angle>-1.57</min_angle>
+                        <max_angle>1.5707</max_angle>
                     </horizontal>
                 </scan>
@@ -1643,7 +1637,7 @@
   <plugin name="gz_ros2_control::GazeboSimROS2ControlPlugin" filename="gz_ros2_control-system">
     <parameters>$(find rcup_garden)/config/mec_drive_controllers.yaml</parameters>
-    <!-- <ros>
-        <remapping>/mec_cont/odom:=/odom</remapping>
-      </ros> -->
+    <ros>
+        <remapping>/mecanum_drive_controller/odom:=/odom</remapping>
+      </ros>
   </plugin>
 </gazebo>
