Commit message: teleop issue fixed and new warehouse world added

File: urdf/ArmPlate.urdf.xacro (robot description, xacro)
@@ -273,5 +273,4 @@
         <mu2>0.2</mu2>
     </gazebo>
-    <!-- updated part ends -->
 <!-- ************************************************************** LINKS : BASE RELEVANT ENDS ***************************************************************-->
 <!-- ************************************************************** LINKS : ARM RELATED(BASE IRRELEVANT) ******************************************************-->
@@ -1151,5 +1150,5 @@
         <parent link="Wheel_motor_2" />
         <child link="wheel2" />
-        <axis xyz="1.0 2.635647389719074e-60 2.139937261679685e-14" />
+        <axis xyz="-1.0 2.635647389719074e-60 2.139937261679685e-14" />
         <limit effort="1000" velocity="1000"/>
         <dynamics damping="1.0" friction="1.0"/>
@@ -1175,5 +1174,5 @@
         <parent link="Wheel_motor_3" />
         <child link="wheel3" />
-        <axis xyz="1.0 -8.619515182870853e-61 2.139937261679685e-14" />
+        <axis xyz="-1.0 -8.619515182870853e-61 2.139937261679685e-14" />
         <limit effort="1000" velocity="1000"/>
         <dynamics damping="1.0" friction="1.0"/>
@@ -1642,8 +1641,8 @@
 <gazebo>
   <plugin name="gz_ros2_control::GazeboSimROS2ControlPlugin" filename="gz_ros2_control-system">
-    <parameters>$(find rcup_garden)/config/mec_drive_controllers.yaml</parameters>
+    <parameters>$(find rcup_garden)/config/diff_drive_controllers.yaml</parameters>
     <!-- <ros>
         <remapping>/mec_cont/odom:=/odom</remapping>
-      </ros> -->
+    </ros> -->
   </plugin>
 </gazebo>

Commit message: Added IMU plugin and bridge for it to get on ROS2 topic

File: urdf/ArmPlate.urdf.xacro (robot description, xacro)
@@ -1545,4 +1545,20 @@
     <!-- GAZEBO PLUGIN FOR LIDAR ENDS -->
 <!-- ************************************************************** LIDAR RELATED LINKS,JOINTS,PLUGINS ENDS****************************************************************-->
+<!-- ************************************************************** IMU RELATED LINKS,JOINTS,PLUGINS ****************************************************************-->
+    <link name="imu_link"/>
+    <joint name="base_final_to_imu" type="fixed">
+      <origin xyz="0 0 0.05" rpy="0 0 0"/> <!-- adjust z offset as needed -->
+      <parent link="base_final-v3"/>
+      <child  link="imu_link"/>
+    </joint>
+    <gazebo reference="imu_link">
+      <sensor name="imu_sensor" type="imu">
+        <always_on>1</always_on>
+        <update_rate>1</update_rate>
+        <visualize>true</visualize>
+        <topic>imu</topic>
+      </sensor>
+    </gazebo>
+<!-- ************************************************************** IMU RELATED LINKS,JOINTS,PLUGINS ENDS****************************************************************-->
 <!-- *************************************************************ROS2 CONTROL TAG ******************************************************************************************** -->
 <!-- ROS 2 Control hardware configuration for mecanum drive -->

Commit message: Mapping is better after the chagnes

File: urdf/ArmPlate.urdf.xacro (robot description, xacro)
@@ -167,13 +167,18 @@
         </visual>
         <collision name="wheel1_collision">
-            <origin xyz="-0.029999999999998934 3.985414700480305e-09 -1.795055695197334e-09" rpy="1.5707963267948986 -3.7599466882338544e-14 1.5707963267949" />
-            <geometry>
-                <mesh filename="file:///home/sanjay/ros2_workspaces/rcup_migration/src/rcup_garden/meshes/Component53.stl" scale="0.001 0.001 0.001" />
+            <origin xyz="0 0 0" rpy="0 1.5708 0" />
+            <geometry>
+                <cylinder radius="0.075" length="0.06"/>
             </geometry>
         </collision>
     </link>
     <gazebo reference="wheel1">
-        <mu1>0.2</mu1>
-        <mu2>0.2</mu2>
+        <mu1>1.0</mu1>
+        <mu2>0.2</mu2>
+        <kp>10000.0</kp>
+        <kd>1.0</kd>
+        <minDepth>0.001</minDepth>
+        <maxVel>0.1</maxVel>
+        <fdir1>1 0 0</fdir1>
     </gazebo>
     <link name="wheel2">
@@ -193,13 +198,18 @@
         </visual>
         <collision name="wheel2_collision">
-            <origin xyz="-0.1474172325407498 0.45000000398542617 0.24999999820496066" rpy="1.5707963267948948 1.5707963267948533 0" />
-            <geometry>
-                <mesh filename="file:///home/sanjay/ros2_workspaces/rcup_migration/src/rcup_garden/meshes/Component54.stl" scale="0.001 0.001 0.001" />
+            <origin xyz="0 0 0" rpy="0 1.5708 0" />
+            <geometry>
+                <cylinder radius="0.075" length="0.06"/>
             </geometry>
         </collision>
     </link>
     <gazebo reference="wheel2">
-        <mu1>0.2</mu1>
-        <mu2>0.2</mu2>
+        <mu1>1.0</mu1>
+        <mu2>0.2</mu2>
+        <kp>10000.0</kp>
+        <kd>1.0</kd>
+        <minDepth>0.001</minDepth>
+        <maxVel>0.1</maxVel>
+        <fdir1>1 0 0</fdir1>
     </gazebo>
     <link name="wheel3">
@@ -219,13 +229,18 @@
         </visual>
         <collision name="wheel3_collision">
-            <origin xyz="-0.014999999999999538 -0.3786419912148507 3.955438074854101e-09" rpy="1.5707963267948983 -3.6508851011130416e-14 1.570796326794899" />
-            <geometry>
-                <mesh filename="file:///home/sanjay/ros2_workspaces/rcup_migration/src/rcup_garden/meshes/Component55.stl" scale="0.001 0.001 0.001" />
+            <origin xyz="0 0 0" rpy="0 1.5708 0" />
+            <geometry>
+                <cylinder radius="0.075" length="0.06"/>
             </geometry>
         </collision>
     </link>
     <gazebo reference="wheel3">
-        <mu1>0.2</mu1>
-        <mu2>0.2</mu2>
+        <mu1>1.0</mu1>
+        <mu2>0.2</mu2>
+        <kp>10000.0</kp>
+        <kd>1.0</kd>
+        <minDepth>0.001</minDepth>
+        <maxVel>0.1</maxVel>
+        <fdir1>1 0 0</fdir1>
     </gazebo>
     <link name="wheel4">
@@ -245,13 +260,18 @@
         </visual>
         <collision name="wheel4_collision">
-            <origin xyz="-0.02999999999999993 3.985434258169108e-09 -1.79505596165086e-09" rpy="1.5707963267948946 1.5707963267948528 0" />
-            <geometry>
-                <mesh filename="file:///home/sanjay/ros2_workspaces/rcup_migration/src/rcup_garden/meshes/Component56.stl" scale="0.001 0.001 0.001" />
+            <origin xyz="0 0 0" rpy="0 1.5708 0" />
+            <geometry>
+                <cylinder radius="0.075" length="0.06"/>
             </geometry>
         </collision>
     </link>
     <gazebo reference="wheel4">
-        <mu1>0.2</mu1>
-        <mu2>0.2</mu2>
+        <mu1>1.0</mu1>
+        <mu2>0.2</mu2>
+        <kp>10000.0</kp>
+        <kd>1.0</kd>
+        <minDepth>0.001</minDepth>
+        <maxVel>0.1</maxVel>
+        <fdir1>1 0 0</fdir1>
     </gazebo>
     <!-- WHEEL LINKS ENDS-->
@@ -1150,5 +1170,5 @@
         <parent link="Wheel_motor_2" />
         <child link="wheel2" />
-        <axis xyz="-1.0 2.635647389719074e-60 2.139937261679685e-14" />
+        <axis xyz="1.0 2.635647389719074e-60 2.139937261679685e-14" />
         <limit effort="1000" velocity="1000"/>
         <dynamics damping="1.0" friction="1.0"/>
@@ -1158,5 +1178,5 @@
         <parent link="Wheel_motor_4" />
         <child link="wheel4" />
-        <axis xyz="-1.0 8.586479331114432e-60 -2.1399372616796854e-14" />
+        <axis xyz="1.0 8.586479331114432e-60 -2.1399372616796854e-14" />
         <limit effort="1000" velocity="1000"/>
         <dynamics damping="1.0" friction="1.0"/>
@@ -1166,5 +1186,5 @@
         <parent link="Wheel_motor_1" />
         <child link="wheel1" />
-        <axis xyz="-1.0 -7.16708135826507e-61 -2.139937261679685e-14" />
+        <axis xyz="1.0 -7.16708135826507e-61 -2.139937261679685e-14" />
         <limit effort="1000" velocity="1000"/>
         <dynamics damping="1.0" friction="1.0"/>
@@ -1174,5 +1194,5 @@
         <parent link="Wheel_motor_3" />
         <child link="wheel3" />
-        <axis xyz="-1.0 -8.619515182870853e-61 2.139937261679685e-14" />
+        <axis xyz="1.0 -8.619515182870853e-61 2.139937261679685e-14" />
         <limit effort="1000" velocity="1000"/>
         <dynamics damping="1.0" friction="1.0"/>
@@ -1602,6 +1622,7 @@
 <!-- ************************************************************** DRIVE PLUGIN ***************************************************************************************** -->
   <!-- To emulate Mecanum wheels in Gazebo with spherical collisions it
-  requires a custom friction model so the vehicle can strafe left to right -->
-  <gazebo reference='wheel2'>
+  requires a custom friction model so the vehicle can strafe left to right
+  ONLY FOR MECANUM WHEELS -->
+  <!-- <gazebo reference='wheel2'>
     <collision>
       <surface>
@@ -1654,5 +1675,5 @@
       </surface>
     </collision>
-  </gazebo>
+  </gazebo> -->
 <gazebo>
   <plugin name="gz_ros2_control::GazeboSimROS2ControlPlugin" filename="gz_ros2_control-system">

Commit message: pinpointed the issue

File: urdf/ArmPlate.urdf.xacro (robot description, xacro)
@@ -279,5 +279,6 @@
     <link name="base_footprint">
         <inertial>
-            <origin xyz="0.0 0.0 0.0" rpy="0.0 0.0 0.0" />
+            <!-- inertial origin set to zero so base_footprint frame sits at its own origin -->
+            <origin xyz="0.0 0.0 0.0" rpy="1.57 0.0 1.57" />
             <mass value="56.0" />
             <inertia ixx="2.5" iyy="2.5" izz="4.5" ixy="0.0" iyz="0.0" ixz="0.0" />
@@ -285,5 +286,6 @@
     </link>
     <joint name="base_to_robot" type="fixed">
-        <origin xyz="0.0 0.35 -0.07" rpy="1.57 0.0 1.57" />
+        <!-- Place base_footprint at the geometric center of the robot (no offset) -->
+        <origin xyz="0.0 0.0 0.0" rpy="1.57 0.0 1.57" />
         <parent link="base_footprint" />
         <child link="base_final-v3" />

Commit message: better position of base_footprint

File: urdf/ArmPlate.urdf.xacro (robot description, xacro)
@@ -280,5 +280,5 @@
         <inertial>
             <!-- inertial origin set to zero so base_footprint frame sits at its own origin -->
-            <origin xyz="0.0 0.0 0.0" rpy="1.57 0.0 1.57" />
+            <origin xyz="0.36831 0.0 0.0" rpy="1.57 0.0 1.57" />
             <mass value="56.0" />
             <inertia ixx="2.5" iyy="2.5" izz="4.5" ixy="0.0" iyz="0.0" ixz="0.0" />
@@ -287,5 +287,5 @@
     <joint name="base_to_robot" type="fixed">
         <!-- Place base_footprint at the geometric center of the robot (no offset) -->
-        <origin xyz="0.0 0.0 0.0" rpy="1.57 0.0 1.57" />
+        <origin xyz="-0.36 0.0 -0.15" rpy="1.57 0.0 1.57" />
         <parent link="base_footprint" />
         <child link="base_final-v3" />

Commit message: set the base_footprint inertial to zero

File: urdf/ArmPlate.urdf.xacro (robot description, xacro)
@@ -278,10 +278,9 @@
     <!-- Updated part for correcting bot orientation on spawn -->
     <link name="base_footprint">
-        <inertial>
-            <!-- inertial origin set to zero so base_footprint frame sits at its own origin -->
+        <!-- <inertial>
             <origin xyz="0.36831 0.0 0.0" rpy="1.57 0.0 1.57" />
             <mass value="56.0" />
             <inertia ixx="2.5" iyy="2.5" izz="4.5" ixy="0.0" iyz="0.0" ixz="0.0" />
-        </inertial>
+        </inertial> -->
     </link>
     <joint name="base_to_robot" type="fixed">
